File: zen/zen.kicad_pcb (KiCad board)
At the start: 2 copper layers, 285.9 x 94.7 mm, 102 parts, among them SW1 SW_Push, SW10 SW_Push, SW11 SW_Push, SW12 SW_Push, SW13 SW_Push, SW14 SW_Push, SW15 SW_Push, SW16 SW_Push, SW17 SW_Push, SW18 SW_Push, SW19 SW_Push, SW2 SW_Push, SW20 SW_Push, SW21 SW_Push, SW22 SW_Push, SW23 SW_Push, SW24 SW_Push, SW25 SW_Push, SW26 SW_Push, SW27 SW_Push, SW28 SW_Push, SW29 SW_Push, SW3 SW_Push, SW30 SW_Push, SW31 SW_Push, SW32 SW_Push, SW33 SW_Push, SW34 SW_Push, SW35 SW_Push, SW36 SW_Push, SW37 SW_Push, SW38 SW_Push, SW4 SW_Push, SW5 SW_Push, SW6 SW_Push, SW7 SW_Push, SW8 SW_Push, SW9 SW_Push, U1 ProMicro, U2 ProMicro

Commit message: pcb complete
Parts:
- U1, U2: value ProMicro -> kb2040
- moved D35 62.9 mm to (118.1, 162.6), turned to 15 degrees
- moved SW35 58.2 mm to (120.2, 168.6), turned to 15 degrees
- moved D38 42.7 mm to (180.9, 170.6), turned to -30 degrees
- moved D37 42.7 mm to (160.8, 162.3), turned to -15 degrees
- moved SW38 39.5 mm to (178.1, 176.2), turned to -30 degrees
- moved SW37 39.5 mm to (159.7, 168.4), turned to -15 degrees
- moved D36 21.4 mm to (139.6, 159.7), turned to 0 degrees
- moved SW36 19.8 mm to (140.0, 165.9), turned to 0 degrees
Connections:
- D20 pad 1: Row0 -> Row0_L
- D21 pad 1: Row0 -> Row0_L
- D22 pad 1: Row0 -> Row0_L
- D23 pad 1: Row0 -> Row0_L
- D24 pad 1: Row0 -> Row0_L
- D25 pad 1: Row1 -> Row1_L
- D26 pad 1: Row1 -> Row1_L
- D27 pad 1: Row1 -> Row1_L
- D28 pad 1: Row1 -> Row1_L
- D29 pad 1: Row1 -> Row1_L
- D30 pad 1: Row2 -> Row2_L
- D31 pad 1: Row2 -> Row2_L
- D32 pad 1: Row2 -> Row2_L
- D33 pad 1: Row2 -> Row2_L
- D34 pad 1: Row2 -> Row2_L
- D35 pad 1: Row3 -> Row3_L
- D36 pad 1: Row3 -> Row3_L
- D37 pad 1: Row3 -> Row3_L
- D38 pad 1: Row3 -> Row3_L
- U1 pad 19: Row0 -> Row3
- U1 pad 20: Row1 -> Row2
- U1 pad 21: Row2 -> Row1
- U1 pad 22: Row3 -> Row0
- U2 pad 19: Row0 -> Row3_L
- U2 pad 20: Row1 -> Row2_L
- U2 pad 21: Row2 -> Row1_L
- U2 pad 22: Row3 -> Row0_L
Routing:
- net ENC1_A: track 0.00 -> 201.3 mm, vias 0 -> 5
- net ENC2_A: track 0.00 -> 201.0 mm, vias 0 -> 2
- net ENC2_B: track 0.00 -> 200.8 mm, vias 0 -> 2
- net ENC1_B: track 0.00 -> 197.1 mm, vias 0 -> 5
- net Col0_L: track 0.00 -> 170.4 mm, vias 0 -> 8
- net Col1_L: track 0.00 -> 167.5 mm, vias 0 -> 6
- net Col3: track 0.00 -> 156.4 mm, vias 0 -> 1
- net Row3: track 0.00 -> 155.9 mm, vias 0 -> 2
- net Col4: track 0.00 -> 153.2 mm, vias 0 -> 1
- net Row2: track 0.00 -> 153.0 mm
- net Row0_L: track 0.00 -> 151.2 mm, vias 0 -> 10
- net Col2_L: track 0.00 -> 149.6 mm, vias 0 -> 4
- net Col2: track 0.00 -> 141.7 mm, vias 0 -> 1
- net Row2_L: track 0.00 -> 137.7 mm
- net Row1: track 0.00 -> 134.2 mm, vias 0 -> 2
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- added copper zone on B.Cu, net GND
- added copper zone on F.Cu, net GND
