File: zen/zen.kicad_sch (KiCad schematic)
At the start: 84 parts, among them SW1 SW_Push, SW10 SW_Push, SW11 SW_Push, SW12 SW_Push, SW13 SW_Push, SW14 SW_Push, SW15 SW_Push, SW16 SW_Push, SW17 SW_Push, SW18 SW_Push, SW19 SW_Push, SW2 SW_Push, SW20 SW_Push, SW21 SW_Push, SW22 SW_Push, SW23 SW_Push, SW24 SW_Push, SW25 SW_Push, SW26 SW_Push, SW27 SW_Push, SW28 SW_Push, SW29 SW_Push, SW3 SW_Push, SW30 SW_Push, SW31 SW_Push, SW32 SW_Push, SW33 SW_Push, SW34 SW_Push, SW35 SW_Push, SW36 SW_Push, SW37 SW_Push, SW38 SW_Push, SW4 SW_Push, SW5 SW_Push, SW6 SW_Push, SW7 SW_Push, SW8 SW_Push, SW9 SW_Push, U1 kb2040, U2 kb2040

Commit message: pcb complete
Connections:
- net Row0: now also U1.22 (A0/26); no longer D20.1 (K), D21.1 (K), D22.1 (K), D23.1 (K), D24.1 (K), U1.19 (A3/29), U2.19 (A3/29)
- net Row1: now also U1.21 (A1/27); no longer D25.1 (K), D26.1 (K), D27.1 (K), D28.1 (K), D29.1 (K), U1.20 (A2/28), U2.20 (A2/28)
- net Row2: now also U1.20 (A2/28); no longer D30.1 (K), D31.1 (K), D32.1 (K), D33.1 (K), D34.1 (K), U1.21 (A1/27), U2.21 (A1/27)
- net Row3: now also U1.19 (A3/29); no longer D35.1 (K), D36.1 (K), D37.1 (K), D38.1 (K), U1.22 (A0/26), U2.22 (A0/26)
- new net Row0_L: D20.1 (K), D21.1 (K), D22.1 (K), D23.1 (K), D24.1 (K), U2.22 (A0/26)
- new net Row1_L: D25.1 (K), D26.1 (K), D27.1 (K), D28.1 (K), D29.1 (K), U2.21 (A1/27)
- new net Row2_L: D30.1 (K), D31.1 (K), D32.1 (K), D33.1 (K), D34.1 (K), U2.20 (A2/28)
- new net Row3_L: D35.1 (K), D36.1 (K), D37.1 (K), D38.1 (K), U2.19 (A3/29)
